Commit message: camera work

File: src/robotDiff/robot_diff_description/urdf/robot_diff.urdf (robot description, URDF)
Before this commit: robot robot_diff, 8 links, 7 joints
Joints:
- joint base_to_camera: origin xyz=0 -0.216 0.151 rpy=0 0 1.571 -> xyz=0 -0.284 0.151 rpy=0 0 4.712
- joint base_to_chassis: origin xyz=0 0 0 rpy=0 0 0 -> xyz=0 0 0 rpy=0 0 3.1415
- joint base_to_lidar: origin xyz=0 -0.25 0.051 rpy=0 0 0 -> xyz=0 -0.25 0.051 rpy=0 0 3.1415
